File: daq_griffin/adc_chain.kicad_sch (KiCad schematic)
At the start: 8 parts, among them U29 REF6050xDGK, U30 TLV70933

Commit message: Inductor footprint changed, ADC fuse value now 30mA, ADC 25R resistor now 22R, 0.1-0.47R resistor set to 0.47R
Parts:
- C110: value 0.1uF -> 100nF
Changed lines of the file:
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@@
 			)
 		)
-		(property "Value" "0.1uF"
+		(property "Value" "100nF"
 			(at 87.63 126.9999 0)
 			(effects

Commit message: Added JLCPCB part numbers to all back side components to be in PCBA
Parts:
- C107: LCSC (none) -> C1592
- C108: LCSC (none) -> C16780
- C110, C111, C112: LCSC (none) -> C1590
- R103: LCSC (none) -> C15401
- U29: LCSC (none) -> C2157003
- U30: LCSC (none) -> C133791
Changed lines of the file:
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@@
+			)
+		)
+		(property "LCSC" "C1590"
+			(at 152.4 142.24 0)
+			(effects
+				(font
+					(size 1.27 1.27)
+				)
+				(hide yes)
 			)
 		)
@@
 		)
 		(property "MPN" "generic R%f %v %r"
+			(at 52.07 156.21 90)
+			(effects
+				(font
+					(size 1.27 1.27)
+				)
+				(hide yes)
+			)
+		)
+		(property "LCSC" "C15401"
 			(at 52.07 156.21 90)
 			(effects
@@
 			)
 		)
+		(property "LCSC" "C1590"
+			(at 114.3 142.24 0)
+			(effects
+				(font
+					(size 1.27 1.27)
+				)
+				(hide yes)
+			)
+		)
 		(pin "1"
 		)
@@
 			)
 		)
+		(property "LCSC" "C1592"
+			(at 40.64 154.94 0)
+			(effects
+				(font
+					(size 1.27 1.27)
+				)
+				(hide yes)
+			)
+		)
 		(pin "1"
 		)
@@
 			)
 		)
+		(property "LCSC" "C1590"
+			(at 83.82 125.73 0)
+			(effects
+				(font
+					(size 1.27 1.27)
+				)
+				(hide yes)
+			)
+		)
 		(pin "1"
 		)
@@
 			)
 		)
+		(property "LCSC" "C133791"
+			(at 134.62 134.62 0)
+			(effects
+				(font
+					(size 1.27 1.27)
+				)
+				(hide yes)
+			)
+		)
 		(pin "1"
 		)
@@
 			)
 		)
+		(property "LCSC" "C2157003"
+			(at 66.04 142.24 0)
+			(effects
+				(font
+					(size 1.27 1.27)
+				)
+				(hide yes)
+			)
+		)
 		(pin "1"
 		)
@@
 			(at 88.9 156.21 0)
 			(effects
+				(font
+					(size 1.27 1.27)
+				)
+				(hide yes)
+			)
+		)
+		(property "LCSC" "C16780"
+			(at 88.9 156.21 0)
+			(effects
